Commit message: added camera naem according to rs_launch.py for consistency!

File: xarm_description/urdf/camera/realsense.gazebo.xacro (robot description, xacro)
@@ -1,5 +1,5 @@
 <?xml version="1.0"?>
 <robot xmlns:xacro="http://ros.org/wiki/xacro">
-  <xacro:macro name="realsense_gazebo" params="prefix:='' ">
+  <xacro:macro name="realsense_gazebo" params="prefix:='' camera_name:='wrist_mounted'">
     <!-- <gazebo reference="${prefix}camera_depth_frame">
       <sensor name="cameradepth" type="depth">
@@ -122,6 +122,6 @@
       </plugin>
     </gazebo> -->
-    <gazebo reference="${prefix}camera_color_frame">
-      <sensor name="${prefix}_rgbd_sensor" type="rgbd_camera">
+    <gazebo reference="${prefix}${camera_name}_camera_color_frame">
+      <sensor name="${prefix}${camera_name}__rgbd_sensor" type="rgbd_camera">
         <camera>
           <horizontal_fov>1.047</horizontal_fov>
@@ -171,11 +171,11 @@
             </clip>
           </depth_camera>
-          <optical_frame_id>${prefix}camera_color_optical_frame</optical_frame_id>
+          <optical_frame_id>${prefix}${camera_name}_camera_color_optical_frame</optical_frame_id>
         </camera>
-        <ignition_frame_id>${prefix}camera_color_frame</ignition_frame_id>
+        <ignition_frame_id>${prefix}${camera_name}_camera_color_frame</ignition_frame_id>
         <always_on>1</always_on>
         <update_rate>10.0</update_rate>
         <visualize>false</visualize>
-        <topic>wrist_mounted_camera</topic>
+        <topic>${camera_name}_camera</topic>
         <enable_metrics>false</enable_metrics>
       </sensor>

File: xarm_description/urdf/camera/realsense_d435i.urdf.xacro (robot description, xacro)
@@ -1,5 +1,5 @@
 <?xml version="1.0"?>
 <robot xmlns:xacro="http://ros.org/wiki/xacro">
-  <xacro:macro name="d435i_urdf" params="prefix:='' add_d435i_links:=false">
+  <xacro:macro name="d435i_urdf" params="prefix:='' camera_name:='wrist_mounted' add_d435i_links:=false">
     <!-- define property -->
     <xacro:property name="M_PI" value="3.1415926535897931" />
@@ -16,56 +16,56 @@
     </link>
     <xacro:if value="${add_d435i_links}">
-      <link name="${prefix}camera_link"></link>
-      <link name="${prefix}camera_depth_frame"></link>
-      <link name="${prefix}camera_depth_optical_frame"></link>
-      <link name="${prefix}camera_color_frame"></link>
-      <link name="${prefix}camera_color_optical_frame"></link>
-      <link name="${prefix}camera_left_ir_frame"></link>
-      <link name="${prefix}camera_left_ir_optical_frame"></link>
-      <link name="${prefix}camera_right_ir_frame"></link>
-      <link name="${prefix}camera_right_ir_optical_frame"></link>
-      <joint name="${prefix}camera_link_joint" type="fixed">
+      <link name="${prefix}${camera_name}_camera_link"></link>
+      <link name="${prefix}${camera_name}_camera_depth_frame"></link>
+      <link name="${prefix}${camera_name}_camera_depth_optical_frame"></link>
+      <link name="${prefix}${camera_name}_camera_color_frame"></link>
+      <link name="${prefix}${camera_name}_camera_color_optical_frame"></link>
+      <link name="${prefix}${camera_name}_camera_left_ir_frame"></link>
+      <link name="${prefix}${camera_name}_camera_left_ir_optical_frame"></link>
+      <link name="${prefix}${camera_name}_camera_right_ir_frame"></link>
+      <link name="${prefix}${camera_name}_camera_right_ir_optical_frame"></link>
+      <joint name="${prefix}${camera_name}_camera_link_joint" type="fixed">
         <parent link="${prefix}link_eef" />
-        <child link="${prefix}camera_link" />
+        <child link="${prefix}${camera_name}_camera_link" />
         <origin xyz="0.06746 -0.0175 0.0237" rpy="${M_PI} ${-M_PI/2} 0" />
       </joint>
-      <joint name="${prefix}camera_depth_joint" type="fixed">
-        <parent link="${prefix}camera_link" />
-        <child link="${prefix}camera_depth_frame" />
+      <joint name="${prefix}${camera_name}_camera_depth_joint" type="fixed">
+        <parent link="${prefix}${camera_name}_camera_link" />
+        <child link="${prefix}${camera_name}_camera_depth_frame" />
         <origin xyz="0 0 0" rpy="0 0 0" />
       </joint>
-      <joint name="${prefix}camera_depth_optical_joint" type="fixed">
-        <parent link="${prefix}camera_depth_frame" />
-        <child link="${prefix}camera_depth_optical_frame" />
+      <joint name="${prefix}${camera_name}_camera_depth_optical_joint" type="fixed">
+        <parent link="${prefix}${camera_name}_camera_depth_frame" />
+        <child link="${prefix}${camera_name}_camera_depth_optical_frame" />
         <origin xyz="0 0 0" rpy="${-M_PI/2} 0 ${-M_PI/2}" />
       </joint>
-      <joint name="${prefix}camera_color_joint" type="fixed">
-        <parent link="${prefix}camera_link" />
-        <child link="${prefix}camera_color_frame" />
+      <joint name="${prefix}${camera_name}_camera_color_joint" type="fixed">
+        <parent link="${prefix}${camera_name}_camera_link" />
+        <child link="${prefix}${camera_name}_camera_color_frame" />
         <origin xyz="0 0.015 0" rpy="0 0 0" />
       </joint>
-      <joint name="${prefix}camera_color_optical_joint" type="fixed">
-        <parent link="${prefix}camera_color_frame" />
-        <child link="${prefix}camera_color_optical_frame" />
+      <joint name="${prefix}${camera_name}_camera_color_optical_joint" type="fixed">
+        <parent link="${prefix}${camera_name}_camera_color_frame" />
+        <child link="${prefix}${camera_name}_camera_color_optical_frame" />
         <origin xyz="0 0 0" rpy="${-M_PI/2} 0 ${-M_PI/2}" />
       </joint>
-      <joint name="${prefix}camera_left_ir_joint" type="fixed">
-        <parent link="${prefix}camera_link" />
-        <child link="${prefix}camera_left_ir_frame" />
+      <joint name="${prefix}${camera_name}_camera_left_ir_joint" type="fixed">
+        <parent link="${prefix}${camera_name}_camera_link" />
+        <child link="${prefix}${camera_name}_camera_left_ir_frame" />
         <origin xyz="0 0 0" rpy="0 0 0" />
       </joint>
-      <joint name="${prefix}camera_left_ir_optical_joint" type="fixed">
-        <parent link="${prefix}camera_left_ir_frame" />
-        <child link="${prefix}camera_left_ir_optical_frame" />
+      <joint name="${prefix}${camera_name}_camera_left_ir_optical_joint" type="fixed">
+        <parent link="${prefix}${camera_name}_camera_left_ir_frame" />
+        <child link="${prefix}${camera_name}_camera_left_ir_optical_frame" />
         <origin xyz="0 0 0" rpy="${-M_PI/2} 0 ${-M_PI/2}" />
       </joint>
-      <joint name="${prefix}camera_right_ir_joint" type="fixed">
-        <parent link="${prefix}camera_link" />
-        <child link="${prefix}camera_right_ir_frame" />
+      <joint name="${prefix}${camera_name}_camera_right_ir_joint" type="fixed">
+        <parent link="${prefix}${camera_name}_camera_link" />
+        <child link="${prefix}${camera_name}_camera_right_ir_frame" />
         <origin xyz="0 -0.050 0" rpy="0 0 0" />
       </joint>
-      <joint name="${prefix}camera_right_ir_optical_joint" type="fixed">
-        <parent link="${prefix}camera_right_ir_frame" />
-        <child link="${prefix}camera_right_ir_optical_frame" />
+      <joint name="${prefix}${camera_name}_camera_right_ir_optical_joint" type="fixed">
+        <parent link="${prefix}${camera_name}_camera_right_ir_frame" />
+        <child link="${prefix}${camera_name}_camera_right_ir_optical_frame" />
         <origin xyz="0 0 0" rpy="${-M_PI/2} 0 ${-M_PI/2}" />
       </joint>
