Commit message: added joint_velocity_cotnroller as mecanum won;t work

File: xarm_description/urdf/uf850/uf850.ros2_control.xacro (robot description, xacro)
@@ -1,5 +1,6 @@
 <?xml version="1.0"?>
 <robot xmlns:xacro="http://ros.org/wiki/xacro">
-  <xacro:macro name="uf850_ros2_control" params="prefix
+  <xacro:macro name="uf850_ros2_control"
+    params="prefix
     velocity_control:='false'
     ros2_control_plugin:='uf_robot_hardware/UFRobotSystemHardware'
@@ -137,4 +138,39 @@
         <!-- <state_interface name="effort"/> -->
       </joint>
+      <!-- <hardware>
+              <plugin>gz_ros2_control/GazeboSimSystem</plugin>
+            </hardware> -->
+      <joint name="joint_wheel_front_left">
+        <command_interface name="velocity">
+          <param name="min">-1</param>
+          <param name="max">1</param>
+        </command_interface>
+        <state_interface name="position" />
+        <state_interface name="velocity" />
+      </joint>
+      <joint name="joint_wheel_front_right">
+        <command_interface name="velocity">
+          <param name="min">-1</param>
+          <param name="max">1</param>
+        </command_interface>
+        <state_interface name="position" />
+        <state_interface name="velocity" />
+      </joint>
+      <joint name="joint_wheel_back_left">
+        <command_interface name="velocity">
+          <param name="min">-1</param>
+          <param name="max">1</param>
+        </command_interface>
+        <state_interface name="position" />
+        <state_interface name="velocity" />
+      </joint>
+      <joint name="joint_wheel_back_right">
+        <command_interface name="velocity">
+          <param name="min">-1</param>
+          <param name="max">1</param>
+        </command_interface>
+        <state_interface name="position" />
+        <state_interface name="velocity" />
+      </joint>
     </ros2_control>
   </xacro:macro>

Commit message: removed base joints from arm joints control

File: xarm_description/urdf/uf850/uf850.ros2_control.xacro (robot description, xacro)
@@ -141,4 +141,5 @@
               <plugin>gz_ros2_control/GazeboSimSystem</plugin>
             </hardware> -->
+<!--
       <joint name="joint_wheel_front_left">
         <command_interface name="velocity">
@@ -172,5 +173,5 @@
         <state_interface name="position" />
         <state_interface name="velocity" />
-      </joint>
+      </joint> -->
     </ros2_control>
   </xacro:macro>

Commit message: added ros2 state interface for topic-based FT sensor

File: xarm_description/urdf/uf850/uf850.ros2_control.xacro (robot description, xacro)
@@ -139,47 +139,11 @@
       </joint>
       <sensor name="force_torque_sensor">
-        <state_interface name="force.x" />
-        <state_interface name="force.y" />
-        <state_interface name="force.z" />
-        <state_interface name="torque.x" />
-        <state_interface name="torque.y" />
-        <state_interface name="torque.z" />
+          <state_interface name="force.x"/>
+          <state_interface name="force.y"/>
+          <state_interface name="force.z"/>
+          <state_interface name="torque.x"/>
+          <state_interface name="torque.y"/>
+          <state_interface name="torque.z"/>
       </sensor>
-      <!-- <hardware>
-              <plugin>gz_ros2_control/GazeboSimSystem</plugin>
-            </hardware> -->
-      <!--
-      <joint name="joint_wheel_front_left">
-        <command_interface name="velocity">
-          <param name="min">-1</param>
-          <param name="max">1</param>
-        </command_interface>
-        <state_interface name="position" />
-        <state_interface name="velocity" />
-      </joint>
-      <joint name="joint_wheel_front_right">
-        <command_interface name="velocity">
-          <param name="min">-1</param>
-          <param name="max">1</param>
-        </command_interface>
-        <state_interface name="position" />
-        <state_interface name="velocity" />
-      </joint>
-      <joint name="joint_wheel_back_left">
-        <command_interface name="velocity">
-          <param name="min">-1</param>
-          <param name="max">1</param>
-        </command_interface>
-        <state_interface name="position" />
-        <state_interface name="velocity" />
-      </joint>
-      <joint name="joint_wheel_back_right">
-        <command_interface name="velocity">
-          <param name="min">-1</param>
-          <param name="max">1</param>
-        </command_interface>
-        <state_interface name="position" />
-        <state_interface name="velocity" />
-      </joint> -->
     </ros2_control>
   </xacro:macro>

Commit message: enable initial pose reading from hivebotics_description

File: xarm_description/urdf/uf850/uf850.ros2_control.xacro (robot description, xacro)
@@ -13,4 +13,6 @@
     joint5_lower_limit:=${-2.1642}  joint5_upper_limit:=${2.1642}
     joint6_lower_limit:=${-2.0*pi}  joint6_upper_limit:=${2.0*pi}">
+    <xacro:property name="initial_positions_file" value="$(find hivebotics_description)/config/initial_positions.yaml"/>
+    <xacro:property name="initial_positions" value="${xacro.load_yaml(initial_positions_file)}"/>
     <ros2_control name="${prefix}${ros2_control_plugin}" type="system">
       <hardware>
@@ -46,5 +48,5 @@
         </command_interface>
         <state_interface name="position">
-          <param name="initial_value">0.0</param>
+          <param name="initial_value">${initial_positions['uf850']['joint1']}</param>
         </state_interface>
         <state_interface name="velocity">
@@ -63,5 +65,9 @@
         </command_interface>
         <state_interface name="position">
+<<<<<<< Updated upstream
           <param name="initial_value">0.035</param>
+=======
+          <param name="initial_value">${initial_positions['uf850']['joint2']}</param>
+>>>>>>> Stashed changes
         </state_interface>
         <state_interface name="velocity">
@@ -80,5 +86,5 @@
         </command_interface>
         <state_interface name="position">
-          <param name="initial_value">-0.0</param>
+          <param name="initial_value">${initial_positions['uf850']['joint3']}</param>
         </state_interface>
         <state_interface name="velocity">
@@ -97,5 +103,5 @@
         </command_interface>
         <state_interface name="position">
-          <param name="initial_value">-0.0</param>
+          <param name="initial_value">${initial_positions['uf850']['joint4']}</param>
         </state_interface>
         <state_interface name="velocity">
@@ -114,5 +120,5 @@
         </command_interface>
         <state_interface name="position">
-          <param name="initial_value">-0.0</param>
+          <param name="initial_value">${initial_positions['uf850']['joint5']}</param>
         </state_interface>
         <state_interface name="velocity">
@@ -131,5 +137,5 @@
         </command_interface>
         <state_interface name="position">
-          <param name="initial_value">0.0</param>
+          <param name="initial_value">${initial_positions['uf850']['joint6']}</param>
         </state_interface>
         <state_interface name="velocity">
