Commit message: Add FDCC compliance controller config and seat-lift sim hooks

File: xarm_description/urdf/common/common.gazebo.xacro (robot description, xacro)
@@ -6,4 +6,7 @@
         <xacro:if value="${ros2_control_params != ''}">
           <parameters>${ros2_control_params}</parameters>
+        </xacro:if>
+        <xacro:if value="${'$(optenv SIM_SCENARIO)' == 'seat_lift'}">
+          <parameters>$(find hivebotics_description)/config/seat_lift_compliance.yaml</parameters>
         </xacro:if>
         <!-- <controller_manager_node_name>${prefix}controller_manager</controller_manager_node_name> -->

File: xarm_description/urdf/uf850/uf850.ros2_control.xacro (robot description, xacro)
@@ -13,5 +13,6 @@
     joint5_lower_limit:=${-2.1642}  joint5_upper_limit:=${2.1642}
     joint6_lower_limit:=${-2.0*pi}  joint6_upper_limit:=${2.0*pi}">
-    <xacro:property name="initial_positions_file" value="$(find hivebotics_description)/config/initial_positions.yaml"/>
+    <xacro:property name="start_pose_file" value="$(optenv SEAT_LIFT_START_POSE_FILE)"/>
+    <xacro:property name="initial_positions_file" value="${start_pose_file if start_pose_file else '$(find hivebotics_description)/config/initial_positions.yaml'}"/>
     <xacro:property name="initial_positions" value="${xacro.load_yaml(initial_positions_file)}"/>
     <ros2_control name="${prefix}${ros2_control_plugin}" type="system">
